Commit message: 更新异构车队地图、导航与 CBS 调度项目

File: src/hetero_fleet_description/urdf/heavy_diff_amr.xacro (robot description, xacro)
@@ -2,13 +2,14 @@
 <!-- Heavy differential-drive AMR for pallet transport.
      SCALE: like the other two robots this is the warehouse design times `s`,
-     which is 0.45 here - NOT the 0.53 that MAP_SWAP.md's table still quotes.
-     The code is the source of truth: s=0.31 gives a 0.409 x 0.267 m body
-     (0.428 x 0.322 m including the bumper, wheels included), and the
+     which is 0.34 here - NOT the 0.53 that MAP_SWAP.md's table still quotes.
+     The code is the source of truth: s=0.34 gives a 0.449 x 0.292 m body
+     (0.469 x 0.354 m including the bumper, wheels included), and the
      controller geometry in heavy_diff_amr_controllers.yaml (wheel_radius
-     0.062 / separation 0.2945) was derived from exactly that. It started at
-     0.45 and has been shrunk twice since (0.36, now 0.31); see the note in
-     light_diff_amr.xacro. Masses scale as s^3, inertias as s^5, and the
+     0.068 / separation 0.323) was derived from exactly that. It started at
+     0.45, was shrunk twice (0.36, then 0.31), and was scaled back up to 0.34
+     on 2026-09-28; see the note in light_diff_amr.xacro.
+     Masses scale as s^3, inertias as s^5, and the
      shell mesh by s, so geometry, dynamics and visuals stay consistent.
-     The navigation footprint in robot_profiles.yaml (0.428 x 0.322 m) is
+     The navigation footprint in robot_profiles.yaml (0.469 x 0.354 m) is
      this same outline, measured by tools/measure_footprint.py.
 -->
@@ -19,5 +20,5 @@
   <xacro:property name="controllers_file" value="$(arg controllers_file)"/>
   <xacro:property name="robot_name" value="$(arg robot_name)"/>
-  <xacro:property name="s" value="0.31"/>
+  <xacro:property name="s" value="0.445526037015"/>
   <xacro:property name="base_length" value="${1.32 * s}"/>
   <xacro:property name="base_width" value="${0.86 * s}"/>
@@ -75,4 +76,16 @@
   <link name="front_caster_link"><visual><geometry><sphere radius="${0.20 * s}"/></geometry><material name="rubber"><color rgba="0.04 0.04 0.04 1"/></material></visual><collision><geometry><sphere radius="${0.20 * s}"/></geometry></collision></link>
   <joint name="front_caster_joint" type="fixed"><parent link="heavy_caster_fork_link"/><child link="front_caster_link"/><origin xyz="0 0 ${-0.02 * s}"/></joint>
+  <!-- Normally clear of the floor by 0.02*s. This rear safety caster
+       arrests backward tipping before the guards touch down and unload the
+       drive wheels. Unlike a fourth coplanar support it does not carry weight
+       during normal driving or compete with the front caster. -->
+  <link name="rear_safety_caster_link">
+    <visual><geometry><sphere radius="${0.18 * s}"/></geometry><material name="rubber"><color rgba="0.04 0.04 0.04 1"/></material></visual>
+    <collision><geometry><sphere radius="${0.18 * s}"/></geometry></collision>
+  </link>
+  <joint name="rear_safety_caster_joint" type="fixed">
+    <parent link="base_link"/><child link="rear_safety_caster_link"/>
+    <origin xyz="${-0.48 * s} 0 0"/>
+  </joint>
   <link name="lidar_link">
     <inertial><mass value="0.18"/><inertia ixx="0.0003" ixy="0" ixz="0" iyy="0.0003" iyz="0" izz="0.0004"/></inertial>
@@ -91,4 +104,5 @@
   <xacro:fleet_gazebo_wheel_dynamics link="right_wheel_link" mu1="1.5" mu2="1.5" kp="10000" kd="100.0" fdir1="1 0 0"/>
   <xacro:fleet_gazebo_wheel_dynamics link="front_caster_link" mu1="0.0" mu2="0.0" kp="10000" kd="100.0"/>
+  <xacro:fleet_gazebo_wheel_dynamics link="rear_safety_caster_link" mu1="0.0" mu2="0.0" kp="10000" kd="100.0"/>
   <xacro:fleet_ros2_control name="${robot_name}" wheel_joints="${['left_wheel_joint', 'right_wheel_joint']}" controller_type="diff" controllers_file="${controllers_file}" namespace="${robot_name}"/>
 </robot>

File: src/hetero_fleet_description/urdf/light_diff_amr.xacro (robot description, xacro)
@@ -2,16 +2,16 @@
 <!-- Lightweight differential-drive AMR, sized for the scanned office map.
      SCALE: every dimension below is the warehouse design multiplied by `s`,
-     which is 0.60 here - NOT the 0.70 that MAP_SWAP.md's table still quotes.
-     The code is the source of truth: s=0.41 gives a 0.328 x 0.221 m body
-     (0.344 x 0.271 m including the bumper, wheels included), which is what
-     the controller geometry (wheel_radius 0.0451 / separation 0.246) and
-     tools/measure_footprint.py report. It started at 0.60 and has been
-     shrunk twice since (0.48, now 0.41): the ring corridor's narrowest
-     usable passage is ~1.1 m and every centimetre of robot width is
-     lateral room the controller gets to work with (see MAP_SWAP.md 3). Masses scale with volume (s^3)
+     which is 0.45 here - NOT the 0.70 that MAP_SWAP.md's table still quotes.
+     The code is the source of truth: s=0.45 gives a 0.360 x 0.243 m body
+     (0.378 x 0.297 m including the bumper, wheels included), which is what
+     the controller geometry (wheel_radius 0.0495 / separation 0.270) and
+     tools/measure_footprint.py report. History: it started at 0.60, was
+     shrunk to 0.48 and then 0.41 to fit the narrow corridor, and was scaled
+     back up to 0.45 on 2026-09-28 at the user's request ("make the robots a
+     bit bigger"). Masses scale with volume (s^3)
      and inertias with s^5, so the dynamics stay self-consistent; the shell
      mesh is scaled by the same factor so the visuals match the collision
      geometry.
-     The navigation footprint in robot_profiles.yaml (0.344 x 0.271 m) is
+     The navigation footprint in robot_profiles.yaml (0.378 x 0.297 m) is
      this same outline, measured by tools/measure_footprint.py.
 -->
@@ -22,5 +22,5 @@
   <xacro:property name="controllers_file" value="$(arg controllers_file)"/>
   <xacro:property name="robot_name" value="$(arg robot_name)"/>
-  <xacro:property name="s" value="0.41"/>
+  <xacro:property name="s" value="0.589666813697"/>
   <xacro:property name="base_length" value="${0.80 * s}"/>
   <xacro:property name="base_width" value="${0.54 * s}"/>

File: src/hetero_fleet_description/urdf/omni_mecanum_amr.xacro (robot description, xacro)
@@ -1,14 +1,15 @@
 <?xml version="1.0"?>
 <!-- Mecanum AMR for precise lateral docking.
-     SCALE: the warehouse design times `s`, which is 0.42 here. The code is the
-     source of truth: s=0.42 gives a 0.378 x 0.294 m body (0.403 x 0.353 m
+     SCALE: the warehouse design times `s`, which is 0.46 here. The code is the
+     source of truth: s=0.46 gives a 0.414 x 0.322 m body (0.442 x 0.386 m
      including the bumper, wheels included), and the controller geometry in
-     omni_mecanum_amr_controllers.yaml (wheels_radius 0.0399, wheel joints at
-     x = +/-0.147, y = +/-0.1617) was derived from exactly that. It started at
-     0.61 and has been shrunk twice since (0.49, now 0.42); see the note in
-     light_diff_amr.xacro. Masses scale as s^3, inertias as s^5, the shell
+     omni_mecanum_amr_controllers.yaml (wheels_radius 0.0437, wheel joints at
+     x = +/-0.161, y = +/-0.177) was derived from exactly that. It started at
+     0.61, was shrunk twice (0.49, then 0.42), and was scaled back up to 0.46
+     on 2026-09-28; see the note in light_diff_amr.xacro.
+     Masses scale as s^3, inertias as s^5, the shell
      mesh by s. The mecanum friction model - which is what makes this robot the
      only one that can strafe - is unchanged; only its dimensions move.
-     The navigation footprint in robot_profiles.yaml (0.403 x 0.353 m) is
+     The navigation footprint in robot_profiles.yaml (0.442 x 0.386 m) is
      this same outline, measured by tools/measure_footprint.py.
 -->
@@ -19,5 +20,5 @@
   <xacro:property name="controllers_file" value="$(arg controllers_file)"/>
   <xacro:property name="robot_name" value="$(arg robot_name)"/>
-  <xacro:property name="s" value="0.42"/>
+  <xacro:property name="s" value="0.602770520669"/>
   <xacro:property name="base_length" value="${0.90 * s}"/>
   <xacro:property name="base_width" value="${0.70 * s}"/>
